File: Eagle/Pyro_Cut-Down.sch (EAGLE design)
At the start: 44 parts, among them IC1 ERIC9-FCC, IC2 MCP111T-240E/TT, IC3 SN74LVC2G02DCTR, IC4 MPL3115A2LGA8, Q1 DMG3415U-7, Q2 2N2222

Commit message: Major update for V2
Major update for V2 of the PCB. Now includes a u-blox CAM-M8Q to provide accurate altitude data. Trigger-at-altitude is now possible.
Parts:
- removed R11: 1K, microbuilder:RESISTOR_0603_NOOUT
- removed R12: 10K, microbuilder:RESISTOR_0603_NOOUT
- added C6: 100nF, microbuilder:CAP_CERAMIC0603_NO
- added IC5: SPX3819-3.3, microbuilder:VREG_SOT23-5
- added Q3: 2N2222, transistor:MMBT2222ALT1-NPN-SOT23-BEC
- added R10: 100K, rcl:R-EU_R0603
- C1: value 1uF -> 10uF; device microbuilder:CAP_CERAMIC0603_NO -> microbuilder:CAP_CERAMIC0805-NOOUTLINE
- C4: device microbuilder:CAP_CERAMIC0603_NO -> rcl:C-EUC0603
- C5: value 10uF -> 10µF
- IC2: value MCP111T-240E/TT -> SN74LVC2G02DCTR; device Microchip-MCP11:MCP111T-270E/TT -> SamacSys_Parts:SN74LVC2G02DCTR; MPN MCP111T-240E/TT -> (none)
- IC3: value SN74LVC2G02DCTR -> CAM-M8; device SamacSys_Parts:SN74LVC2G02DCTR -> ubloxLib:CAM-M8
- IC4: value MPL3115A2LGA8 -> MCP111T-240E/TT; device SparkFun-Sensors:MPL3115A2LGA8 -> Microchip-MCP11:MCP111T-270E/TT; MPN (none) -> MCP111T-240E/TT
- Q2: value 2N2222 -> DMG3415U-7; device transistor:MMBT2222ALT1-NPN-SOT23-BEC -> microbuilder:MOSFET-PWIDE
- R1: value 2.2K -> 1K
- R3: value 100k -> 10K
- R5: value 1K -> 10K
- R6: value 100K -> 1K
- R7: value 1K -> 100k
- R8: value 1K -> 100K
- R9: value 10K -> 2.2K
Connections:
- removed net N$25: C2.1, IC4.CAP
- removed net RESET: IC1.RESET, IC2.VOUT, RESET.2
- removed net VBAT: BAT1.+, D2.A, Q1.S, R9.1
- new net !RESET: IC1.RESET, IC3.!RESET, IC4.VOUT, RESET.2
- new net +3V3: C5.1, C6.1, IC3.V_BCKP, IC5.OUT, Q2.S, R10.1
- new net 3V3SW: C4.1, IC3.VCC, IC3.VCC_IO, Q2.D
- new net N$8: IC3.RF_IN, IC3.RF_OUT
- new net PIN1: IC1.CD, R7.2, R8.1
- new net V+: BAT1.+, D2.A, Q1.S, R5.1
- net FIRE: now also IC2.2Y, R3.1, R4.1; no longer IC3.2Y, R11.1, R12.1
- net GND: now also C6.2, IC2.GND, IC3.GND$1, IC3.GND$10, IC3.GND$11, IC3.GND$12, IC3.GND$13, IC3.GND$14, IC3.GND$2, IC3.GND$3, IC3.GND$4, IC3.GND$5, IC3.GND$6, IC3.GND$7, IC3.GND$8, IC3.GND$9, IC4.VSS, IC5.GND, Q3.E, R3.2, R8.2; no longer IC2.VSS, IC3.GND, IC4.GND, Q2.E, R12.2, R6.2
- net N$19: now also Q3.C, R5.2; no longer Q2.C, R9.2
- net N$2: now also R6.2; no longer R7.2
- net N$20: now also Q3.B, R4.2; no longer Q2.B, R11.2
- net N$4: now also R9.2; no longer R1.2
- net N$5: now also R1.1; no longer R5.1
- net N$6: now also IC2.1Y, IC2.2B; no longer IC3.1Y, IC3.2B
- net N$7: now also R2.1; no longer R8.1
- net PIN15: now also Q2.G, R10.2; no longer C1.1, IC4.VDD, IC4.VDDIO, R2.1, R4.1
- net PIN16: now also R6.1; no longer R7.1
- net PIN17: now also IC2.VCC; no longer IC3.VCC
- net PIN18: now also IC2.1A, IC2.1B; no longer IC3.1A, IC3.1B
- net PIN19: now also IC2.2A; no longer IC3.2A
- net PIN20: now also IC3.TXD/SPI_MISO; no longer IC4.SCL, R2.2
- net PIN21: now also IC3.RXD/SPI_MOSI; no longer IC4.SDA, R4.2
- net PIN22: no longer R3.2, R6.1
- net PYRO: now also R7.1, R9.1; no longer R1.1, R3.1
- net RTS: now also R2.2; no longer R8.2
- net TXD: now also R1.2; no longer R5.2
- net VCC: now also C1.1, C2.1, IC4.VDD, IC5.EN, IC5.IN; no longer C4.1, C5.1, IC2.VDD
Other:
- note added: "Pyro Balloon Cut-Down V2"
- note added: "u-blox CAM-M8"
- note removed: "0x60"
- note removed: "0xC0"
- note removed: "0xC1"
- note removed: "Pyro Balloon Cut-Down V1"
- note removed: "Read Address:"
- note removed: "Slave Address:"
- note removed: "VCC = 3.6V Max"
- note removed: "Write Address:"
